File: proyectos_esquematico_kicad/esquematico_lcd/esquematico_lcd.kicad_pcb (KiCad board)
At the start: 2 copper layers, 2 parts, among them J1 Conn_01x14_Male, U1 RC1602A

Commit message: Se agrega routeo LCD PCB
Parts:
- J1: moved to B.Cu
- U1: footprint Displays:RC1602A -> Display:WC1602A
- moved U1 84.7 mm to (109.9, 51.3)
- moved J1 69.9 mm to (114.3, 62.2)
Connections:
- J1 pad 1: RS -> Net-(J1-Pad1)
- J1 pad 10: DB6 -> POT
- J1 pad 11: DB7 -> DB6
- J1 pad 12: Net-(J1-Pad12) -> VCC
- J1 pad 13: VCC -> DB7
- J1 pad 3: E -> RS
- J1 pad 5: Net-(J1-Pad5) -> E
- J1 pad 7: POT -> DB4
- J1 pad 8: DB4 -> Net-(J1-Pad8)
Routing:
- net GND: track 0.00 -> 71.1 mm
- net VCC: track 0.00 -> 63.7 mm
- net POT: track 0.00 -> 31.0 mm
- net DB6: track 0.00 -> 20.1 mm
- net DB5: track 0.00 -> 19.9 mm
- net DB4: track 0.00 -> 19.9 mm
- net DB7: track 0.00 -> 19.4 mm
- net E: track 0.00 -> 12.2 mm
- net RS: track 0.00 -> 11.2 mm
Other:
- board outline added: 44.5 x 25.4 mm
- rule pad_to_mask_clearance: 0.051 -> 0
- rule trace_min: 0.4064 -> 0.2

Commit message: Cambios menores al PCB del LCD
Routing:
- net VCC: track 63.7 -> 72.1 mm
- net GND: track 71.1 -> 73.7 mm, vias 0 -> 2
- added copper zone on B.Cu, net GND
- added copper zone on F.Cu, net GND
Other:
- net class Default: clearance 0.6096 -> 1.096
- rule trace_clearance: 0.6096 -> 1.096
Changed lines of the file:
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@@
-(kicad_pcb (version 20171130) (host pcbnew 5.1.4-e60b266~84~ubuntu16.04.1)
+(kicad_pcb (version 20171130) (host pcbnew 5.1.5-52549c5~84~ubuntu16.04.1)
   (general
     (thickness 1.6)
-    (drawings 8)
-    (tracks 58)
+    (drawings 9)
+    (tracks 66)
     (zones 0)
     (modules 2)
@@
   )
   (setup
-    (last_trace_width 0.508)
+    (last_trace_width 1.016)
     (user_trace_width 1.016)
     (user_trace_width 1.27)
-    (trace_clearance 0.6096)
+    (trace_clearance 1.096)
     (zone_clearance 0.508)
     (zone_45_only no)
@@
   (net 18 "Net-(J1-Pad8)")
   (net_class Default "This is the default net class."
-    (clearance 0.6096)
+    (clearance 1.096)
     (trace_width 0.508)
     (via_dia 1.778)
@@
     )
   )
+  (dimension 44.45 (width 0.15) (layer B.SilkS)
+    (gr_text "44,450 mm" (at 130.175 77.499999) (layer B.SilkS)
+      (effects (font (size 1 1) (thickness 0.15)))
+    )
+    (feature1 (pts (xy 152.4 71.755) (xy 152.4 76.78642)))
+    (feature2 (pts (xy 107.95 71.755) (xy 107.95 76.78642)))
+    (crossbar (pts (xy 107.95 76.199999) (xy 152.4 76.199999)))
+    (arrow1a (pts (xy 152.4 76.199999) (xy 151.273496 76.78642)))
+    (arrow1b (pts (xy 152.4 76.199999) (xy 151.273496 75.613578)))
+    (arrow2a (pts (xy 107.95 76.199999) (xy 109.076504 76.78642)))
+    (arrow2b (pts (xy 107.95 76.199999) (xy 109.076504 75.613578)))
+  )
   (gr_line (start 152.4 71.12) (end 137.16 71.12) (layer Edge.Cuts) (width 0.1))
   (gr_line (start 152.4 55.88) (end 152.4 71.12) (layer Edge.Cuts) (width 0.1))
@@
   (segment (start 119.38 60.96) (end 119.38 62.23) (width 1.016) (layer F.Cu) (net 3))
   (segment (start 122.575001 57.764999) (end 119.38 60.96) (width 1.016) (layer F.Cu) (net 3))
-  (segment (start 114.955001 57.836117) (end 114.955001 51.320001) (width 1.016) (layer B.Cu) (net 6))
-  (segment (start 111.76 66.04) (end 111.76 61.031118) (width 1.016) (layer B.Cu) (net 6))
-  (segment (start 124.46 64.77) (end 124.46 65.991314) (width 1.016) (layer B.Cu) (net 6))
-  (segment (start 124.46 65.991314) (end 123.141314 67.31) (width 1.016) (layer B.Cu) (net 6))
-  (segment (start 123.141314 67.31) (end 113.03 67.31) (width 1.016) (layer B.Cu) (net 6))
-  (segment (start 111.76 61.031118) (end 114.955001 57.836117) (width 1.016) (layer B.Cu) (net 6))
-  (segment (start 113.03 67.31) (end 111.76 66.04) (width 1.016) (layer B.Cu) (net 6))
+  (segment (start 113.115551 67.237601) (end 111.832399 65.954449) (width 1.016) (layer F.Cu) (net 6))
+  (segment (start 114.955001 53.636001) (end 114.955001 51.320001) (width 1.016) (layer F.Cu) (net 6))
+  (segment (start 123.213713 67.237601) (end 113.115551 67.237601) (width 1.016) (layer F.Cu) (net 6))
+  (segment (start 124.46 65.991314) (end 123.213713 67.237601) (width 1.016) (layer F.Cu) (net 6))
+  (segment (start 124.46 64.77) (end 124.46 65.991314) (width 1.016) (layer F.Cu) (net 6))
+  (segment (start 114.955001 53.636001) (end 114.955001 56.494999) (width 1.016) (layer F.Cu) (net 6))
+  (segment (start 111.832399 65.954449) (end 112.156475 66.278525) (width 1.016) (layer F.Cu) (net 6))
+  (segment (start 111.832399 59.617601) (end 111.832399 65.954449) (width 1.016) (layer F.Cu) (net 6))
+  (segment (start 114.955001 56.494999) (end 111.832399 59.617601) (width 1.016) (layer F.Cu) (net 6))
   (segment (start 135.275001 53.636001) (end 135.275001 51.320001) (width 1.016) (layer F.Cu) (net 7))
   (segment (start 121.92 62.23) (end 121.92 61.008686) (width 1.016) (layer F.Cu) (net 7))
@@
   (segment (start 142.895001 53.954999) (end 142.895001 51.320001) (width 1.016) (layer F.Cu) (net 10))
   (segment (start 134.62 62.23) (end 142.895001 53.954999) (width 1.016) (layer F.Cu) (net 10))
-  (segment (start 127 65.991314) (end 128.318686 67.31) (width 1.016) (layer B.Cu) (net 11))
-  (segment (start 145.435001 53.636001) (end 145.435001 51.320001) (width 1.016) (layer B.Cu) (net 11))
-  (segment (start 131.761002 67.31) (end 145.435001 53.636001) (width 1.016) (layer B.Cu) (net 11))
-  (segment (start 128.318686 67.31) (end 131.761002 67.31) (width 1.016) (layer B.Cu) (net 11))
-  (segment (start 112.415001 51.320001) (end 112.415001 57.764999) (width 1.016) (layer B.Cu) (net 11))
-  (segment (start 110.13439 60.04561) (end 110.13439 66.95439) (width 1.016) (layer B.Cu) (net 11))
-  (segment (start 112.415001 57.764999) (end 110.13439 60.04561) (width 1.016) (layer B.Cu) (net 11))
-  (segment (start 127 65.991314) (end 127 64.77) (width 1.016) (layer B.Cu) (net 11))
-  (segment (start 124.055704 68.93561) (end 127 65.991314) (width 1.016) (layer B.Cu) (net 11))
-  (segment (start 112.11561 68.93561) (end 124.055704 68.93561) (width 1.016) (layer B.Cu) (net 11))
-  (segment (start 110.13439 66.95439) (end 112.11561 68.93561) (width 1.016) (layer B.Cu) (net 11))
-  (segment (start 120.035001 53.636001) (end 120.035001 51.320001) (width 1.016) (layer B.Cu) (net 12))
-  (segment (start 121.009 54.61) (end 120.035001 53.636001) (width 1.016) (layer B.Cu) (net 12))
-  (segment (start 128.27 54.61) (end 121.009 54.61) (width 1.016) (layer B.Cu) (net 12))
+  (segment (start 127 66.438147) (end 124.088536 69.349611) (width 1.016) (layer F.Cu) (net 11))
+  (segment (start 127 64.77) (end 127 66.438147) (width 1.016) (layer F.Cu) (net 11))
+  (segment (start 124.088536 69.349611) (end 112.240728 69.349611) (width 1.016) (layer F.Cu) (net 11))
+  (segment (start 112.240728 69.349611) (end 109.720389 66.829272) (width 1.016) (layer F.Cu) (net 11))
+  (segment (start 109.720389 66.829272) (end 109.720389 57.284611) (width 1.016) (layer F.Cu) (net 11))
+  (segment (start 112.415001 54.589999) (end 112.415001 51.320001) (width 1.016) (layer F.Cu) (net 11))
+  (segment (start 109.720389 57.284611) (end 112.415001 54.589999) (width 1.016) (layer F.Cu) (net 11))
+  (segment (start 145.435001 53.636001) (end 145.435001 51.320001) (width 1.016) (layer F.Cu) (net 11))
+  (segment (start 145.435001 64.114999) (end 145.435001 53.636001) (width 1.016) (layer F.Cu) (net 11))
+  (segment (start 142.312399 67.237601) (end 145.435001 64.114999) (width 1.016) (layer F.Cu) (net 11))
+  (segment (start 127 64.77) (end 127 65.991314) (width 1.016) (layer F.Cu) (net 11))
+  (segment (start 127 65.991314) (end 128.246287 67.237601) (width 1.016) (layer F.Cu) (net 11))
+  (segment (start 128.246287 67.237601) (end 142.312399 67.237601) (width 1.016) (layer F.Cu) (net 11))
   (segment (start 129.54 64.77) (end 130.761314 64.77) (width 1.016) (layer B.Cu) (net 12))
   (segment (start 130.761314 64.77) (end 132.08 63.451314) (width 1.016) (layer B.Cu) (net 12))
   (segment (start 132.08 63.451314) (end 132.08 58.42) (width 1.016) (layer B.Cu) (net 12))
-  (segment (start 132.08 58.42) (end 128.27 54.61) (width 1.016) (layer B.Cu) (net 12))
   (segment (start 109.875001 49.004001) (end 109.875001 51.320001) (width 1.016) (layer B.Cu) (net 12))
   (segment (start 120.035001 51.320001) (end 120.035001 48.915001) (width 1.016) (layer B.Cu) (net 12))
@@
   (segment (start 147.975001 51.320001) (end 147.975001 49.004001) (width 1.016) (layer B.Cu) (net 12))
   (segment (start 147.231 48.26) (end 119.38 48.26) (width 1.016) (layer B.Cu) (net 12))
+  (segment (start 120.035001 53.636001) (end 120.035001 51.320001) (width 1.016) (layer B.Cu) (net 12))
+  (segment (start 121.009 54.61) (end 120.035001 53.636001) (width 1.016) (layer B.Cu) (net 12))
+  (segment (start 128.27 54.61) (end 121.009 54.61) (width 1.016) (layer B.Cu) (net 12))
+  (segment (start 132.08 58.42) (end 128.27 54.61) (width 1.016) (layer B.Cu) (net 12))
+  (via (at 141.605 60.96) (size 1.778) (drill 0.9906) (layers F.Cu B.Cu) (net 12))
+  (via (at 139.7 63.5) (size 1.778) (drill 0.9906) (layers F.Cu B.Cu) (net 12))
+  (segment (start 129.54 64.77) (end 131.445 64.77) (width 1.016) (layer F.Cu) (net 12))
+  (segment (start 131.445 64.77) (end 132.08 64.77) (width 1.016) (layer F.Cu) (net 12))
+  (zone (net 12) (net_name GND) (layer F.Cu) (hatch edge 0.508)
+    (connect_pads (clearance 0.508))
+    (min_thickness 0.254)
+    (fill yes (arc_segments 32) (thermal_gap 0.508) (thermal_bridge_width 0.508))
+    (polygon
+      (pts
+        (xy 151.765 70.485) (xy 108.585 70.485) (xy 108.585 46.355) (xy 151.765 46.355)
+      )
+    )
+  )
+  (zone (net 12) (net_name GND) (layer B.Cu) (hatch edge 0.508)
+    (connect_pads (clearance 0.508))
+    (min_thickness 0.254)
+    (fill yes (arc_segments 32) (thermal_gap 0.508) (thermal_bridge_width 0.508))
+    (polygon
+      (pts
+        (xy 151.765 70.485) (xy 108.585 70.485) (xy 108.585 46.355) (xy 151.765 46.355)
+      )
+    )
+  )
 )
