File: proyectos_esquematico_kicad/Placa_lcd_cont_geiger/Placa_lcd_cont_geiger.sch (KiCad schematic (older format))
At the start: 18 parts, among them J1 Conn_02x04_Counter_Clockwise, J2 Conn_01x14_Female, J3 Conn_01x05_Female, P1 Power, P2 Analog, P3 Digital, P4 Digital, Q1 BC548, Q2 BC548, Q3 BC558

Commit message: Modificaciones en el PCB para poder mardarlo a hacer al LCI. Agregado del esquematico del Arduino UNO R3 actualizado a la carpeta 'doc'
Parts:
- J3: footprint Connector_JST:JST_XH_B05B-XH-A_1x05_P2.50mm_Vertical -> Connectors_Molex:Molex_KK-6410-05_05x2.54mm_Straight
- Q1, Q2, Q3: footprint Package_TO_SOT_THT:TO-92_Inline -> Package_TO_SOT_THT:TO-92_Inline_Wide
Changed lines of the file:
@@
 EESchema Schematic File Version 4
 LIBS:Placa_lcd_cont_geiger-cache
-EELAYER 26 0
+EELAYER 29 0
 EELAYER END
 $Descr A4 11693 8268
@@
 F 0 "Q1" H 1991 5046 50  0000 L CNN
 F 1 "BC548" H 1991 4955 50  0000 L CNN
-F 2 "Package_TO_SOT_THT:TO-92_Inline" H 2000 4925 50  0001 L CIN
+F 2 "Package_TO_SOT_THT:TO-92_Inline_Wide" H 2000 4925 50  0001 L CIN
 F 3 "http://www.fairchildsemi.com/ds/BC/BC547.pdf" H 1800 5000 50  0001 L CNN
 	1    1800 5000
@@
 F 0 "Q2" H 3400 4500 50  0000 L CNN
 F 1 "BC548" H 3250 4400 50  0000 L CNN
-F 2 "Package_TO_SOT_THT:TO-92_Inline" H 3750 4175 50  0001 L CIN
+F 2 "Package_TO_SOT_THT:TO-92_Inline_Wide" H 3750 4175 50  0001 L CIN
 F 3 "http://www.fairchildsemi.com/ds/BC/BC547.pdf" H 3550 4250 50  0001 L CNN
 	1    3550 4250
@@
 F 0 "Q3" H 3500 4650 50  0000 L CNN
 F 1 "BC558" H 3400 4550 50  0000 L CNN
-F 2 "Package_TO_SOT_THT:TO-92_Inline" H 3900 4725 50  0001 L CIN
+F 2 "Package_TO_SOT_THT:TO-92_Inline_Wide" H 3900 4725 50  0001 L CIN
 F 3 "http://www.fairchildsemi.com/ds/BC/BC557.pdf" H 3700 4800 50  0001 L CNN
 	1    3700 4800
@@
 F 0 "J3" V 3940 3462 50  0000 R CNN
 F 1 "Conn_01x05_Female" V 3849 3462 50  0000 R CNN
-F 2 "Connector_JST:JST_XH_B05B-XH-A_1x05_P2.50mm_Vertical" H 4000 3750 50  0001 C CNN
+F 2 "Connectors_Molex:Molex_KK-6410-05_05x2.54mm_Straight" H 4000 3750 50  0001 C CNN
 F 3 "~" H 4000 3750 50  0001 C CNN
 	1    4000 3750

Commit message: Cambios menores en el shield para adaptarlo a los cambios hechos sobre el prototipo
Parts:
- added R3: 10k, Resistor_THT:R_Axial_DIN0207_L6.3mm_D2.5mm_P10.16mm_Horizontal, symbol Device:R
Connections:
- net A1: now also R2.2
- net A2: now also R1.2
- net A4: no longer R2.2
- net A5: now also R3.2; no longer R1.2
- net at Q3.2 (B), R1.1: no longer Q2.2 (B)
- new net: Q2.2 (B), R3.1
- no-connect marks 25 -> 23
Changed lines of the file:
@@
 EESchema Schematic File Version 4
-LIBS:Placa_lcd_cont_geiger-cache
-EELAYER 29 0
+EELAYER 30 0
 EELAYER END
 $Descr A4 11693 8268
@@
 $EndComp
 NoConn ~ 8950 1450
-NoConn ~ 8900 2600
-NoConn ~ 8900 2700
 NoConn ~ 8900 2800
 NoConn ~ 10550 2900
@@
 $EndComp
 Connection ~ 9300 3150
-Text Label 1100 5000 2    60   ~ 0
-A4
-Text Label 2700 4800 2    60   ~ 0
+Text Label 2700 4250 2    60   ~ 0
 A5
 NoConn ~ 10550 1800
@@
 Wire Wire Line
 	2700 4800 2800 4800
-Wire Wire Line
-	3100 4800 3350 4800
 $Comp
 L power:GND #PWR0101
@@
 	3800 4300 3800 4600
 Wire Wire Line
-	3350 4250 3350 4800
-Connection ~ 3350 4800
-Wire Wire Line
-	3350 4800 3500 4800
-Wire Wire Line
 	4000 3950 4000 4100
 Wire Wire Line
@@
 	4200 4750 4250 4750
 Connection ~ 4250 4750
+Wire Wire Line
+	3100 4800 3500 4800
+$Comp
+L Device:R R3
+U 1 1 5E1FAAA8
+P 3000 4250
+F 0 "R3" V 2793 4250 50  0000 C CNN
+F 1 "10k" V 2884 4250 50  0000 C CNN
+F 2 "Resistor_THT:R_Axial_DIN0207_L6.3mm_D2.5mm_P10.16mm_Horizontal" V 2930 4250 50  0001 C CNN
+F 3 "~" H 3000 4250 50  0001 C CNN
+	1    3000 4250
+	0    1    1    0
+$EndComp
+Wire Wire Line
+	3350 4250 3150 4250
+Text Label 2700 4800 2    60   ~ 0
+A2
+Text Label 1100 5000 2    60   ~ 0
+A1
+Wire Wire Line
+	2850 4250 2700 4250
 $EndSCHEMATC
